Commit message: fix: package paths

File: realsense2_description/urdf_examples/d435.urdf (robot description, URDF)
Before this commit: robot realsense2_camera, 4 links, 3 joints
Links:
- link camera_link: geometry collision box size=0.02505 0.09 0.025; visual mesh filename=package://realsense2_description/meshes/d435.dae

File: realsense2_description/urdf_examples/l515.urdf (robot description, URDF)
Before this commit: robot realsense2_camera, 4 links, 3 joints
Links:
- link camera_link: geometry collision cylinder length=0.026 radius=0.0305; visual mesh filename=package://realsense2_description/meshes/l515.dae
